Commit message: :recycle: refac: adjust URDF parameters for lidar and collision; update ROS-Gazebo bridge configuration

File: src/scout_description/urdf/scout_mini.xacro (robot description, xacro)
@@ -147,5 +147,5 @@
             </geometry>
             <material>
-                <color rgba="0.0 1.0 0.0 1.0" />
+                <color rgba="250.0 0.0 0.0 1.0" />
             </material>
         </visual>
@@ -157,5 +157,5 @@
         <inertial>
             <mass value="0.1" />
-            <origin xyz="0 0 0" />
+            <origin xyz="0 00 0" />
             <inertia ixx="0.001" iyy="0.001" izz="0.001" ixy="0" ixz="0" iyz="0" />
         </inertial>
@@ -164,5 +164,5 @@
         <parent link="base_link" />
         <child link="lidar_link" />
-        <origin xyz="0 0 0.2" rpy="0 0 0" />
+        <origin xyz="0 0 0.05" rpy="0 0 0" />
     </joint>
     <!-- <gazebo reference="lidar_link">
@@ -201,6 +201,6 @@
                     <horizontal>
                         <samples>360</samples>
-                        <min_angle>-3.14</min_angle>
-                        <max_angle>3.14</max_angle>
+                        <min_angle>0</min_angle>
+                        <max_angle>6.28</max_angle>
                     </horizontal>
                 </scan>

Commit message: :bug: fix: adjust lidar parameters and improve wall avoidance logic for better obstacle detection and handling

File: src/scout_description/urdf/scout_mini.xacro (robot description, xacro)
@@ -142,22 +142,24 @@
     <!-- Lidar init-->
     <link name="lidar_link">
-        <visual>
-            <geometry>
-                <cylinder radius="0.05" length="0.02" />
-            </geometry>
-            <material>
-                <color rgba="250.0 0.0 0.0 1.0" />
+        <inertial>
+            <mass value="0.1" />
+            <origin xyz="0 0 0" />
+            <inertia ixx="0.001" iyy="0.001" izz="0.001" ixy="0" ixz="0" iyz="0" />
+        </inertial>
+        <visual>
+            <origin xyz="0 0 0" rpy="0 0 0" />
+            <geometry>
+                <cylinder radius="0.05" length="0.05" />
+            </geometry>
+            <material name="white">
+                <color rgba="1 1 1 1" />
             </material>
         </visual>
         <collision>
-            <geometry>
-                <cylinder radius="0.05" length="0.02" />
-            </geometry>
-        </collision>
-        <inertial>
-            <mass value="0.1" />
-            <origin xyz="0 00 0" />
-            <inertia ixx="0.001" iyy="0.001" izz="0.001" ixy="0" ixz="0" iyz="0" />
-        </inertial>
+            <origin xyz="0 0 0" rpy="0 0 0" />
+            <geometry>
+                <cylinder radius="0.05" length="0.05" />
+            </geometry>
+        </collision>
     </link>
     <joint name="lidar_joint" type="fixed">
@@ -166,30 +168,7 @@
         <origin xyz="0 0 0.05" rpy="0 0 0" />
     </joint>
-    <!-- <gazebo reference="lidar_link">
-        <sensor type="ray" name="lidar_sensor">
-            <update_rate>10</update_rate>
-            <ray>
-                <scan>
-                    <horizontal>
-                        <samples>720</samples>
-                        <resolution>1.0</resolution>
-                        <min_angle>-1.57</min_angle>
-                        <max_angle>1.57</max_angle>
-                    </horizontal>
-                </scan>
-                <range>
-                    <min>0.1</min>
-                    <max>10.0</max>
-                    <resolution>0.01</resolution>
-                </range>
-            </ray>
-            <plugin filename="libgz-sim-sensors-system.so" name="gz::sim::systems::Sensors">
-                <render_engine>ogre2</render_engine>
-            </plugin>
-        </sensor>
-    </gazebo> -->
     <gazebo reference="lidar_link">
         <sensor name="lidar_sensor" type="gpu_lidar">
-            <pose> 0 0 0 0 0 0 </pose>
+            <pose> 0 0 0.02 0 0 0 </pose>
             <always_on>true</always_on>
             <visualize>true</visualize>

Commit message: :rocket: feat: add RGB front camera and 3d lidar to model

File: src/scout_description/urdf/scout_mini.xacro (robot description, xacro)
@@ -148,7 +148,7 @@
         </inertial>
         <visual>
-            <origin xyz="0 0 0" rpy="0 0 0" />
-            <geometry>
-                <cylinder radius="0.05" length="0.05" />
+            <origin xyz="0 0 -0.02" rpy="0 0 0" />
+            <geometry>
+                <cylinder radius="0.05" length="0.1" />
             </geometry>
             <material name="white">
@@ -157,7 +157,7 @@
         </visual>
         <collision>
-            <origin xyz="0 0 0" rpy="0 0 0" />
-            <geometry>
-                <cylinder radius="0.05" length="0.05" />
+            <origin xyz="-0 0 -0.02" rpy="0 0 0" />
+            <geometry>
+                <cylinder radius="0.05" length="0.1" />
             </geometry>
         </collision>
@@ -166,9 +166,9 @@
         <parent link="base_link" />
         <child link="lidar_link" />
-        <origin xyz="0 0 0.05" rpy="0 0 0" />
+        <origin xyz="0 0 0.1" rpy="0 0 0" />
     </joint>
     <gazebo reference="lidar_link">
-        <sensor name="lidar_sensor" type="gpu_lidar">
-            <pose> 0 0 0.02 0 0 0 </pose>
+        <sensor name="lidar_sensor" type="gpu_ray">
+            <pose> 0 0 0 0 0 0 </pose>
             <always_on>true</always_on>
             <visualize>true</visualize>
@@ -183,4 +183,9 @@
                         <max_angle>6.28</max_angle>
                     </horizontal>
+                    <vertical>
+                        <samples>16</samples>
+                        <min_angle>-0.262</min_angle>
+                        <max_angle>0.523</max_angle>
+                    </vertical>
                 </scan>
                 <range>
@@ -192,4 +197,58 @@
     </gazebo>
     <!-- Lidar end-->
+    <!-- RGB cam start-->
+    <link name="camera_link">
+        <inertial>
+            <mass value="0.1" />
+            <origin xyz="0 0 0" />
+            <inertia ixx="0.001" iyy="0.001" izz="0.001" ixy="0" ixz="0" iyz="0" />
+        </inertial>
+        <visual>
+            <origin xyz="0 0 0" rpy="0 0 0" />
+            <geometry>
+                <box size="0.05 0.05 0.05" />
+            </geometry>
+            <material name="white">
+                <color rgba="1 1 1 1" />
+            </material>
+        </visual>
+        <collision>
+            <origin xyz="0 0 0" rpy="0 0 0" />
+            <geometry>
+                <box size="0.05 0.05 0.05" />
+            </geometry>
+        </collision>
+    </link>
+    <joint name="camera_joint" type="fixed">
+        <parent link="base_link" />
+        <child link="camera_link" />
+        <origin xyz="0.18 0 0.05" rpy="0 0 0" />
+    </joint>
+    <gazebo reference="camera_link">
+        <sensor name="rgb_cam" type="camera">
+            <always_on>1</always_on>
+            <update_rate>60</update_rate>
+            <visualize>1</visualize>
+            <pose>0 0.0175 0.5125 0 0 0</pose>
+            <topic>scout_mini/rgb_cam/image_raw</topic>
+            <camera name="rgb_cam">
+                <horizontal_fov>1.21126</horizontal_fov>
+                <image>
+                    <width>640</width>
+                    <height>480</height>
+                    <format>RGB_INT8</format>
+                </image>
+                <clip>
+                    <near>0.1</near>
+                    <far>100</far>
+                </clip>
+                <noise>
+                    <type>gaussian</type>
+                    <mean>0</mean>
+                    <stddev>0.007</stddev>
+                </noise>
+            </camera>
+        </sensor>
+    </gazebo>
     <!-- Scout gazebo plugin -->
     <gazebo>

Commit message: :bug: fix: update README instructions and adjust inertial parameters for correct robot dynamics

File: src/scout_description/urdf/scout_mini.xacro (robot description, xacro)
@@ -22,8 +22,9 @@
         name="inertial_link">
         <inertial>
-            <mass value="132.3898489950015" />
+            <mass value="23" />
             <origin xyz=" 0 0 0" />
-            <inertia ixx="0.185196122711036" ixy="4.30144213829512E-08" ixz="5.81037523686401E-08"
-                iyy="0.364893736238929" iyz="-0.000386720198091934" izz="0.223868521722778" />
+            <!-- <inertia ixx="0.185196122711036" ixy="4.30144213829512E-08" ixz="5.81037523686401E-08"
+                iyy="0.364893736238929" iyz="-0.000386720198091934" izz="0.223868521722778" /> -->
+                <inertia ixx="0.83292392" ixy="0" ixz="0" iyy="0.75981458" iyz="0" izz="1.36264267"/>
         </inertial>
     </link>
@@ -40,5 +41,6 @@
             <mass value="3" />
             <origin xyz="0 0 0" />
-            <inertia ixx="0.7171" ixy="0" ixz="0" iyy="0.7171" iyz="0" izz="0.1361" />
+            <!-- <inertia ixx="0.7171" ixy="0" ixz="0" iyy="0.7171" iyz="0" izz="0.1361" /> -->
+            <inertia ixx="0.00671406" ixy="0" ixz="0" iyy="0.00671406" iyz="0" izz="0.01148438"/>
         </inertial>
         <visual>
@@ -66,5 +68,6 @@
             <mass value="3" />
             <origin xyz="0 0 0" />
-            <inertia ixx="0.7171" ixy="0" ixz="0" iyy="0.7171" iyz="0" izz="0.1361" />
+            <!-- <inertia ixx="0.7171" ixy="0" ixz="0" iyy="0.7171" iyz="0" izz="0.1361" /> -->
+            <inertia ixx="0.00671406" ixy="0" ixz="0" iyy="0.00671406" iyz="0" izz="0.01148438"/>
         </inertial>
         <visual>
@@ -92,5 +95,6 @@
             <mass value="3" />
             <origin xyz="0 0 0" />
-            <inertia ixx="0.7171" ixy="0" ixz="0" iyy="0.7171" iyz="0" izz="0.1361" />
+            <!-- <inertia ixx="0.7171" ixy="0" ixz="0" iyy="0.7171" iyz="0" izz="0.1361" /> -->
+            <inertia ixx="0.00671406" ixy="0" ixz="0" iyy="0.00671406" iyz="0" izz="0.01148438"/>
         </inertial>
         <visual>
@@ -118,5 +122,6 @@
             <mass value="3" />
             <origin xyz="0 0 0" />
-            <inertia ixx="0.7171" ixy="0" ixz="0" iyy="0.7171" iyz="0" izz="0.1361" />
+            <!-- <inertia ixx="0.7171" ixy="0" ixz="0" iyy="0.7171" iyz="0" izz="0.1361" /> -->
+            <inertia ixx="0.00671406" ixy="0" ixz="0" iyy="0.00671406" iyz="0" izz="0.01148438"/>z
         </inertial>
         <visual>
@@ -170,5 +175,5 @@
     <gazebo reference="lidar_link">
         <sensor name="lidar_sensor" type="gpu_ray">
-            <pose> 0 0 0 0 0 0 </pose>
+            <pose> 0 0 0.1 0 0 0 </pose>
             <always_on>true</always_on>
             <visualize>true</visualize>

Commit message: refactor: update MovementParams struct documentation and adjust lidar and camera mass values

File: src/scout_description/urdf/scout_mini.xacro (robot description, xacro)
@@ -148,5 +148,5 @@
     <link name="lidar_link">
         <inertial>
-            <mass value="0.1" />
+            <mass value="0.5" />
             <origin xyz="0 0 0" />
             <inertia ixx="0.001" iyy="0.001" izz="0.001" ixy="0" ixz="0" iyz="0" />
@@ -205,5 +205,5 @@
     <link name="camera_link">
         <inertial>
-            <mass value="0.1" />
+            <mass value="0.3" />
             <origin xyz="0 0 0" />
             <inertia ixx="0.001" iyy="0.001" izz="0.001" ixy="0" ixz="0" iyz="0" />
